File: boost-mult.kicad_pcb.pre-toggle-switch.kicad_pcb (KiCad board)
At the start: 2 copper layers, 19 x 100 mm, 29 parts, among them J1 IN, J2 OUT1, J3 OUT2, J4 OUT3, J5 OUT4, J6 PWR, SW1 AC_COUPLE, SW2 DRIVE, U1 TL074, U2 TL072

Commit message: update switches
Parts:
- SW1, SW2: footprint drichert:ToggleSwitch_1x03_P2.54mm_Vertical -> Button_Switch_THT:SW_Slide_SPDT_Straight_CK_OS102011MS2Q
- moved C5 10.3 mm to (136.0, 94.6), turned to -90 degrees
- moved R3 9.96 mm to (136.0, 98.0), turned to -90 degrees
- moved SW1 4.85 mm to (127.0, 97.5), turned to 90 degrees
- moved SW2 4.85 mm to (132.0, 97.5), turned to 90 degrees
Routing:
- net Net-(SW1-A): track 3.00 -> 17.6 mm, vias 0 -> 2
- net Net-(SW1-C): track 15.5 -> 20.2 mm
- net Net-(SW2-A): track 15.4 -> 11.7 mm
- net Net-(SW2-C): track 48.7 -> 51.9 mm
