File: boost-mult.kicad_sch (KiCad schematic)
At the start: 23 parts, among them J1 IN, J2 OUT1, J3 OUT2, J4 OUT3, J5 OUT4, SW1 AC_COUPLE, SW2 DRIVE, U1 TL074, U2 TL072

Commit message: update switches
Parts:
- SW1, SW2: footprint Button_Switch_THT:SW_Slide_SPDT_Straight_CK_OS102011MS2Q -> drichert:ToggleSwitch_1x03_P2.54mm_Vertical
Changed lines of the file:
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@@
 			)
 		)
-		(property "Footprint" "Button_Switch_THT:SW_Slide_SPDT_Straight_CK_OS102011MS2Q"
+		(property "Footprint" "drichert:ToggleSwitch_1x03_P2.54mm_Vertical"
 			(at 137.16 69.85 0)
 			(effects
@@
 			)
 		)
-		(property "Footprint" "Button_Switch_THT:SW_Slide_SPDT_Straight_CK_OS102011MS2Q"
+		(property "Footprint" "drichert:ToggleSwitch_1x03_P2.54mm_Vertical"
 			(at 167.64 62.23 0)
 			(effects

Commit message: tht film cap, move standoff hole
Parts:
- C5: footprint Capacitor_SMD:C_0805_2012Metric -> Capacitor_THT:C_Rect_L7.2mm_W4.5mm_P5.00mm_FKS2_FKP2_MKS2_MKP2
Changed lines of the file:
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@@
 			)
 		)
-		(property "Footprint" "Capacitor_SMD:C_0805_2012Metric"
+		(property "Footprint" "Capacitor_THT:C_Rect_L7.2mm_W4.5mm_P5.00mm_FKS2_FKP2_MKS2_MKP2"
 			(at 151.13 71.4248 0)
 			(effects
